File: sparkGap2.kicad_sch (KiCad schematic)
At the start: 46 parts, among them J1 9V, J2 IN, J3 OUT, Q1 BS170, SW1 SPST, SW2 6-pin Footswitch, U1 TL072

Commit message: Cleaner PCB layout. Better CNC placement. Added cut guides for pedal sides. Updated build guide.
Parts:
- C1, C2: MFG (none) -> TDK; MFG Part (none) -> B32529C1222K189
- C10, C4, C8: MFG (none) -> Vishay; MFG Part (none) -> MKT1817410065
- C11, C13: footprint Capacitor_THT:CP_Radial_D6.3mm_P2.50mm -> Capacitor_THT:CP_Radial_D5.0mm_P2.00mm; MFG (none) -> Panasonic; MFG Part (none) -> EEU-FR1H220
- C12, C14: MFG (none) -> Rubycon; MFG Part (none) -> 16PX1000MEFC10X12.5
- C3: MFG (none) -> Panasonic; MFG Part (none) -> EEU-FR1H100
- C5, C7: MFG (none) -> TDK; MFG Part (none) -> B32529C1472K000
- C6: MFG (none) -> WIMA; MFG Part (none) -> FKS2D004701A00JSSD
- C9: MFG (none) -> TDK; MFG Part (none) -> B32529C0333K189
- D1: MFG (none) -> onsemi; MFG Part (none) -> 1N4001RLG
- D2, D3: MFG (none) -> American Bright Optoelectronics Corporation; MFG Part (none) -> BL-BJU3V1; Notes (none) -> Choose whatever you want as long as it's a 3mm LED
- D4: MFG (none) -> onsemi; MFG Part (none) -> 1N4148-T50A
- GAIN1, TONE1, VOL.1: MFG (none) -> Alps; MFG Part (none) -> RK09L1140A5L
- J1: MFG (none) -> Tensility; MFG Part (none) -> 54-00151; Notes (none) -> 2.1mm ID, 5.5mm OD. Generic is fine. Must be insulated.; now in the parts list
- J2: MFG (none) -> Neutrik; MFG Part (none) -> NMJ4HC-S; Notes (none) -> This needs to have a switch. Generic is fine
- J3: MFG (none) -> Neutrik; MFG Part (none) -> NMJ4HC-S; Notes (none) -> Switch not necessary. Generic is fine
- Mount1, Mount2: MFG (none) -> Würth; MFG Part (none) -> 971100354; Notes (none) -> 10mm M3 standoffs
- Q1: MFG (none) -> onsemi; MFG Part (none) -> BS170
- R1, R11, R12, R13, R2, R3, R4, R5, R6, R7, R8: Notes (none) -> standard 1/4W generic resistors
- R14: value 1k -> 270; Notes (none) -> standard 1/4W generic resistors. Adjust for LED voltage dro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
- SW1: MFG (none) -> Adam tech; MFG Part (none) -> SW-T3-1A-A-A3-S1; Notes (none) -> on-off switch. Generic fine. Body should be ~0.27"x ~0.52" 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
- SW2: MFG (none) -> Alpha; MFG Part (none) -> SF12020DF; Notes (none) -> DPDT foot switch. Generics work
- U1: MFG (none) -> TI; MFG Part (none) -> TL072IP; Notes (none) -> Avoid generics. Buy TI
Other:
- moved on the sheet: C1, C10, C11, C12, C13, C14, C2, C3, C4, C5, C6, C7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
